Commit message: Move important information into the observation space. Fix gate dimensions to reflect the real setup. Add more docs. Add passive env checker tests.

File: lsy_drone_racing/sim/assets/obstacle.urdf (robot description, URDF)
Before this commit: robot obstacle, 3 links, 2 joints
Links:
- link cylinder_link: geometry collision cylinder length=0.8 radius=0.05; visual cylinder length=1.4 radius=0.05

Commit message: Add collective thrust env to deploy script

File: lsy_drone_racing/sim/assets/obstacle.urdf (robot description, URDF)
Before this commit: robot obstacle, 3 links, 2 joints
Links:
- link cylinder_link: geometry collision cylinder length=1.4 radius=0.05; visual cylinder length=1.4 radius=0.05
